File: Beaks Pro/Hardware/beaks_pro.kicad_pcb (KiCad board)
At the start: 2 copper layers, 126 parts, among them J1 Pins_02x08_P1.27mm_TH, J10 Pins_02x08_P2.54mm_TH, J11 out1, J12 out2, J13 Eurorack Power, J2 Pins_02x08_P1.27mm_TH, J3 CV1, J4 CV2, J5 CV3, J6 CV4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

Commit message: Update PCB from schematics
Parts:
- removed D1, D2: LED, LED_THT:LED_D3.0mm
- removed J10: Pins_02x08_P2.54mm_TH, Connector_PinSocket_2.54mm:PinSocket_2x08_P2.54mm_Vertical
- removed SW1: SW_TRIG2, Button_Switch_THT:SW_PUSH_6mm_H13mm
- removed SW4: SW_TRIG1, Button_Switch_THT:SW_PUSH_6mm_H13mm
- added C24: 100n, Capacitor_THT:C_Rect_L10.0mm_W4.0mm_P7.50mm_MKS4, F.Cu at (219.6, 118.0)
- added H1: MountingHole, MountingHole:MountingHole_2.7mm_M2.5, F.Cu at (264.5, 125.0)
- added H2: MountingHole, MountingHole:MountingHole_2.7mm_M2.5, F.Cu at (249.2, 137.6)
- added J14: Pins_02x10_P2.54mm_TH, Connector_PinHeader_2.54mm:PinHeader_2x10_P2.54mm_Vertical, F.Cu at (240.8, 136.4)
- added R58: 47k, Resistor_THT:R_Axial_DIN0207_L6.3mm_D2.5mm_P7.62mm_Horizontal, F.Cu at (208.3, 113.5)
- added R59: 47k, Resistor_THT:R_Axial_DIN0207_L6.3mm_D2.5mm_P7.62mm_Horizontal, F.Cu at (208.3, 117.6)
- added R60: 100k, Resistor_THT:R_Axial_DIN0207_L6.3mm_D2.5mm_P7.62mm_Horizontal, F.Cu at (208.3, 121.7)
- added R61: 100k, Resistor_THT:R_Axial_DIN0207_L6.3mm_D2.5mm_P7.62mm_Horizontal, F.Cu at (208.3, 125.7)
- added R62: 47k, Resistor_THT:R_Axial_DIN0207_L6.3mm_D2.5mm_P7.62mm_Horizontal, F.Cu at (208.3, 129.8)
- added R63: 47k, Resistor_THT:R_Axial_DIN0207_L6.3mm_D2.5mm_P7.62mm_Horizontal, F.Cu at (208.3, 133.8)
- added R64: 100k, Resistor_THT:R_Axial_DIN0207_L6.3mm_D2.5mm_P7.62mm_Horizontal, F.Cu at (208.3, 137.8)
- added R65: 100k, Resistor_THT:R_Axial_DIN0207_L6.3mm_D2.5mm_P7.62mm_Horizontal, F.Cu at (208.3, 141.9)
- added RV10: B100k, Library:Potentiometer_Alps_RK09K_Single_Vertical, F.Cu at (232.9, 122.5)
- added RV9: B100k, Library:Potentiometer_Alps_RK09K_Single_Vertical, F.Cu at (232.9, 108.1)
- added SW5: SW_ML6, Library:ML6-H2T2GQA, F.Cu at (265.6, 108.0)
- added SW6: SW_ML6, Library:ML6-H2T2GQA, F.Cu at (265.6, 117.0)
- added U9: TL072CP, PCM_Package_DIP_AKL:DIP-8_W7.62mm_Socket_LongPads, F.Cu at (219.6, 105.5)
- J1: value Pins_02x08_P1.27mm_TH -> Pins_02x10_P2.54mm_TH; footprint Connector_PinHeader_2.54mm:PinHeader_2x08_P2.54mm_Vertical -> Connector_PinHeader_2.54mm:PinHeader_2x10_P2.54mm_Vertical
- J2: value Pins_02x08_P1.27mm_TH -> Pins_02x10_P2.54mm_TH; footprint Connector_PinHeader_2.54mm:PinHeader_2x08_P2.54mm_Vertical -> Connector_PinSocket_2.54mm:PinSocket_2x10_P2.54mm_Vertical
- J9: value Pins_02x08_P2.54mm_TH -> Pins_02x10_P2.54mm_TH; footprint Connector_PinSocket_2.54mm:PinSocket_2x08_P2.54mm_Vertical -> Connector_PinSocket_2.54mm:PinSocket_2x10_P2.54mm_Vertical
- RV1, RV2, RV3, RV7: footprint Library:Potentiometer_Alps_RK09K_Single_Vertical -> Library:Potentiometer_Alps_RK09K_Single_Vertical_DSHAFT
- RV4, RV5, RV6, RV8: footprint Library:Potentiometer_Alps_RK09K_Single_Vertical_DSHAFT -> Library:Potentiometer_Alps_RK09K_Single_Vertical
- moved J9 167.5 mm to (258.7, 105.8)
- moved J2 72.1 mm to (251.6, 105.8)
- moved J1 62.0 mm to (233.6, 136.4)
- moved R43 50.3 mm to (208.3, 105.5)
- moved R44 50.3 mm to (208.3, 109.5)
Connections:
- C14 pad 2: Net-(C14-Pad2) -> /PRE_ATV_OUT1
- C15 pad 2: Net-(C15-Pad2) -> /PRE_ATV_OUT2
- J1 pad 1: /CV1_JACK -> /PRE_ATV_OUT1
- J1 pad 10: /CV4_POT -> /SW_TRIG1
- J1 pad 11: /CV2_POT -> /LED2
- J1 pad 12: /CV4_ATVPOT -> /SW_TRIG2
- J1 pad 13: /CV3_JACK -> /LED3
- J1 pad 14: /CV4_JACK -> GND
- J1 pad 15: /CV3_ATVPOT -> /LED4
- J1 pad 16: /CV3_POT -> GND
- J1 pad 2: /-10V_REF -> /PRE_ATV_OUT2
- J1 pad 3: /CV1_ATVPOT -> /OUT1_ATVPOT
- J1 pad 4: GND -> /OUT2_ATVPOT
- J1 pad 5: /CV1_POT -> /LED_SALIDA_1
- J1 pad 6: /TRIG_1 -> /SW_DUAL
- J1 pad 7: /CV2_JACK -> /LED_SALIDA_2
- J1 pad 8: /TRIG_2 -> /SW_MODE
- J1 pad 9: /CV2_ATVPOT -> /LED1
- J2 pad 1: /LED_SALIDA_1 -> GND
- J2 pad 10: GND -> /Front PCB/CV2_JACK
- J2 pad 11: /LED4 -> /Front PCB/CV4_POT
- J2 pad 12: GND -> /Front PCB/CV2_ATVPOT
- J2 pad 13: /LED5 -> /Front PCB/CV4_ATVPOT
- J2 pad 14: /OUT1 -> /Front PCB/CV2_POT
- J2 pad 15: GND -> /Front PCB/CV4_JACK
- J2 pad 16: /OUT2 -> /Front PCB/CV3_JACK
- J2 pad 2: /SW_DUAL -> GND
- J2 pad 3: /LED_SALIDA_2 -> /Front PCB/-10V_REF
- J2 pad 4: /SW_MODE -> /Front PCB/CV1_JACK
- J2 pad 5: /LED1 -> GND
- J2 pad 6: /SW_TRIG1 -> /Front PCB/CV1_ATVPOT
- J2 pad 7: /LED2 -> /Front PCB/TRIG_1
- J2 pad 8: /SW_TRIG2 -> /Front PCB/CV1_POT
- J2 pad 9: /LED3 -> /Front PCB/TRIG_2
- J9 pad 1: /Front PCB/-10V_REF -> /Front PCB/PRE_ATV_OUT2
- J9 pad 10: /Front PCB/CV2_ATVPOT -> /Front PCB/LED1
- J9 pad 11: /Front PCB/CV4_ATVPOT -> /Front PCB/SW_TRIG2
- J9 pad 12: /Front PCB/CV2_POT -> /Front PCB/LED2
- J9 pad 13: /Front PCB/CV4_JACK -> GND
- J9 pad 14: /Front PCB/CV3_JACK -> /Front PCB/LED3
- J9 pad 15: /Front PCB/CV3_POT -> GND
- J9 pad 16: /Front PCB/CV3_ATVPOT -> /Front PCB/LED4
- J9 pad 2: /Front PCB/CV1_JACK -> /Front PCB/PRE_ATV_OUT1
- J9 pad 3: GND1 -> /Front PCB/OUT2_ATVPOT
- J9 pad 4: /Front PCB/CV1_ATVPOT -> /Front PCB/OUT1_ATVPOT
- J9 pad 5: /Front PCB/TRIG_1 -> /Front PCB/SW_DUAL
- J9 pad 6: /Front PCB/CV1_POT -> /Front PCB/LED_SALIDA_1
- J9 pad 7: /Front PCB/TRIG_2 -> /Front PCB/SW_MODE
- J9 pad 8: /Front PCB/CV2_JACK -> /Front PCB/LED_SALIDA_2
- J9 pad 9: /Front PCB/CV4_POT -> /Front PCB/SW_TRIG1
- R41 pad 1: Net-(C14-Pad2) -> /PRE_ATV_OUT1
- R42 pad 1: Net-(C15-Pad2) -> /PRE_ATV_OUT2
- R43 pad 2: Net-(C14-Pad2) -> Net-(R43-Pad2)
- R44 pad 2: Net-(C15-Pad2) -> Net-(R44-Pad2)
- U5 pad 1: Net-(C15-Pad2) -> /PRE_ATV_OUT2
- U5 pad 14: Net-(C14-Pad2) -> /PRE_ATV_OUT1

Commit message: Pre-placement on layout, 8HP version
Parts:
- J2, J9: moved to B.Cu
- moved C1 284.5 mm to (395.7, 117.8)
- moved C10 284.5 mm to (474.9, 28.2)
- moved C11 284.5 mm to (474.9, 31.9)
- moved C12 284.5 mm to (474.9, 35.5)
- moved C13 284.5 mm to (481.0, 45.0)
- moved C14 284.5 mm to (474.9, 39.2)
- moved C15 284.5 mm to (474.9, 42.9)
- moved C16 284.5 mm to (463.5, 60.0)
- moved C17 284.5 mm to (455.0, 62.0)
- moved C18 284.5 mm to (455.0, 71.5)
- moved C19 284.5 mm to (455.0, 81.0)
- moved C2 284.5 mm to (395.7, 123.3)
- moved C20 284.5 mm to (463.5, 65.5)
- moved C21 284.5 mm to (463.5, 71.0)
- moved C22 284.5 mm to (463.5, 76.6)
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Other:
- board outline added: 40 x 110 mm
