File: Beaks Pro/Hardware/input.kicad_sch (KiCad schematic)
At the start: 40 parts, among them U1 TL072CP, U2 MCP6002-I-P, U3 TL072CP, U4 MCP6002-I-P

Commit message: 10HP Version
Initial commit with populated PCB for 10HP ver.
Parts:
- removed R1, R15, R16, R17, R18, R2, R3, R4: 47k, Resistor_THT:R_Axial_DIN0207_L6.3mm_D2.5mm_P7.62mm_Horizontal, symbol Device:R
- U1, U2, U3, U4: footprint PCM_Package_DIP_AKL:DIP-8_W7.62mm_Socket_LongPads -> Package_DIP:CERDIP-8_W7.62mm_SideBrazed_LongPads_Socket
Connections:
- net CV1_ATVPOT is gone; now on net GND: U1.3 (+)
- net CV1_JACK is gone; now on net GND: R5.1
- net CV2_ATVPOT is gone; now on net GND: U1.5 (+)
- net CV2_JACK is gone; now on net GND: R6.1
- net CV3_ATVPOT is gone; now on net GND: U3.3 (+)
- net CV3_JACK is gone; now on net GND: R19.1
- net CV4_ATVPOT is gone; now on net GND: U3.5 (+)
- net CV4_JACK is gone; now on net GND: R20.1
