File: Beaks Pro/Hardware/power.kicad_sch (KiCad schematic)
At the start: 17 parts, among them J13 Eurorack Power, U6 LM4040LP-10, U7 L78L05_TO92

Commit message: 10HP Version
Initial commit with populated PCB for 10HP ver.
Parts:
- U7: footprint PCM_Package_TO_SOT_THT_AKL:TO-92L_Inline_Wide -> Package_TO_SOT_THT:TO-92L_Inline_Wide
Changed lines of the file:
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@@
 			)
 		)
-		(property "Footprint" "PCM_Package_TO_SOT_THT_AKL:TO-92L_Inline_Wide"
+		(property "Footprint" "Package_TO_SOT_THT:TO-92L_Inline_Wide"
 			(at 168.91 65.405 0)
 			(effects
