File: Beaks Pro/Hardware/beaks_pro_8hp/input.kicad_sch (KiCad schematic)
At the start: 40 parts, among them U1 TL072CP, U2 MCP6002-I-P, U3 TL072CP, U4 MCP6002-I-P

Commit message: Layout done on 8HP SMT version
Parts:
- added C26: 100n, Capacitor_SMD:C_0603_1608Metric_Pad1.08x0.95mm_HandSolder, symbol Device:C
- C1, C2, C5, C6: footprint Capacitor_THT:C_Rect_L10.0mm_W4.0mm_P7.50mm_MKS4 -> Capacitor_SMD:C_0603_1608Metric_Pad1.08x0.95mm_HandSolder
- C3, C4, C7, C8: footprint Capacitor_THT:C_Disc_D3.4mm_W2.1mm_P2.50mm -> Capacitor_SMD:C_0603_1608Metric_Pad1.08x0.95mm_HandSolder
- R1, R10, R11, R12, R13, R14, R15, R16, R17, R18, R19, R2, R20, R21, R22, R23, R24, R25, R26, R27, R28, R3, R4, R5, R6, R7, R8, R9: footprint Resistor_THT:R_Axial_DIN0207_L6.3mm_D2.5mm_P7.62mm_Horizontal -> Resistor_SMD:R_0603_1608Metric_Pad0.98x0.95mm_HandSolder
- U1, U3: value TL072CP -> TL072CD; footprint PCM_Package_DIP_AKL:DIP-8_W7.62mm_Socket_LongPads -> PCM_Package_SO_AKL:SO-8_3.9x4.9mm_P1.27mm; symbol PCM_Amplifier_Operational_AKL:TL072CP -> PCM_Amplifier_Operational_AKL:TL072CD
- U2, U4: value MCP6002-I-P -> MCP6002-I-SN; footprint PCM_Package_DIP_AKL:DIP-8_W7.62mm_Socket_LongPads -> PCM_Package_SO_AKL:SO-8_3.9x4.9mm_P1.27mm; symbol PCM_Amplifier_Operational_AKL:MCP6002-I-P -> PCM_Amplifier_Operational_AKL:MCP6002-I-SN
Connections:
- net -12V: now also C26.2; no longer C5.2
- net GND: now also C5.2, C26.1
Other:
- moved on the sheet: C5
