File: Beaks Pro/Hardware/beaks_pro_8hp/out.kicad_sch (KiCad schematic)
At the start: 34 parts, among them U5 TL074, U9 TL072CP

Commit message: Layout done on 8HP SMT version
Parts:
- removed unit 5 of U5
- added C25: 100n, Capacitor_SMD:C_0603_1608Metric_Pad1.08x0.95mm_HandSolder, symbol Device:C
- C10, C11, C12, C14, C15, C9: footprint Capacitor_THT:C_Disc_D3.4mm_W2.1mm_P2.50mm -> Capacitor_SMD:C_0603_1608Metric_Pad1.08x0.95mm_HandSolder
- C13, C24: footprint Capacitor_THT:C_Rect_L10.0mm_W4.0mm_P7.50mm_MKS4 -> Capacitor_SMD:C_0603_1608Metric_Pad1.08x0.95mm_HandSolder
- R29, R30, R31, R32, R33, R34, R35, R36, R37, R38, R39, R40, R41, R42, R43, R44, R58, R59, R60, R61, R62, R63, R64, R65: footprint Resistor_THT:R_Axial_DIN0207_L6.3mm_D2.5mm_P7.62mm_Horizontal -> Resistor_SMD:R_0603_1608Metric_Pad0.98x0.95mm_HandSolder
- U5: value TL074 -> TL074CD; footprint Package_DIP:DIP-14_W7.62mm_Socket_LongPads -> PCM_Package_SO_AKL:SOIC-14_3.9x8.7mm_P1.27mm; symbol Amplifier_Operational:TL074 -> PCM_Amplifier_Operational_AKL:TL074CD
- U9: value TL072CP -> TL072CD; footprint PCM_Package_DIP_AKL:DIP-8_W7.62mm_Socket_LongPads -> PCM_Package_SO_AKL:SO-8_3.9x4.9mm_P1.27mm; symbol PCM_Amplifier_Operational_AKL:TL072CP -> PCM_Amplifier_Operational_AKL:TL072CD
Connections:
- net +12V: now also U5.4 (V+)
- net -12V: now also U5.11 (V-), C25.2; no longer C13.2
- net GND: now also C13.2, C25.1
Other:
- moved on the sheet: C13
