File: Beaks Pro/Hardware/beaks_pro_8hp/power.kicad_sch (KiCad schematic)
At the start: 17 parts, among them J13 Eurorack Power, U6 LM4040LP-10, U7 L78L05_TO92

Commit message: Layout done on 8HP SMT version
Parts:
- removed C17, C18, C19: 10u, Capacitor_THT:CP_Radial_D8.0mm_P3.50mm, symbol PCM_Capacitor_AKL:CP_Radial_D8.0mm_P3.50mm
- removed C21: 0,33u, Capacitor_THT:C_Rect_L10.0mm_W4.0mm_P7.50mm_MKS4, symbol PCM_Capacitor_AKL:CP_Radial_D8.0mm_P3.50mm
- removed D10: 3.6, Diode_THT:D_DO-35_SOD27_P7.62mm_Horizontal, symbol Device:D_Zener
- removed U6: LM4040LP-10, Package_TO_SOT_THT:TO-92_Inline_Wide, symbol Reference_Voltage:LM4040LP-10
- removed U7: L78L05_TO92, PCM_Package_TO_SOT_THT_AKL:TO-92L_Inline_Wide, symbol Regulator_Linear:L78L05_TO92
- added C17, C18, C19, C21: 22uF, Capacitor_SMD:C_1206_3216Metric_Pad1.33x1.80mm_HandSolder, symbol Device:C
- added DZ1: ZMM3V6, PCM_Diode_SMD_AKL:D_SOD-323, symbol PCM_Diode_Zener_AKL:MM3Z3V6ST
- added U6: LM4040DBZ-10, Package_TO_SOT_SMD:SOT-23, symbol Reference_Voltage:LM4040DBZ-10
- added U7: AMS1117-5.0, Package_TO_SOT_SMD:SOT-223-3_TabPin2, symbol Regulator_Linear:AMS1117-5.0
- C16, C20, C22: footprint Capacitor_THT:C_Rect_L10.0mm_W4.0mm_P7.50mm_MKS4 -> Capacitor_SMD:C_0603_1608Metric_Pad1.08x0.95mm_HandSolder
- C23: value 100n -> 22uF; footprint Capacitor_THT:C_Rect_L10.0mm_W4.0mm_P7.50mm_MKS4 -> Capacitor_SMD:C_1206_3216Metric_Pad1.33x1.80mm_HandSolder
- D11, D8, D9: value 1N5817 -> B140HW-7; footprint Diode_THT:D_DO-41_SOD81_P10.16mm_Horizontal -> Diode_SMD:D_SOD-123; symbol Diode:1N5817 -> PCM_4ms_Diode:B140HW-7; Alt JLCPCB ID (none) -> C8598; Alt JLCPCB Part (none) -> B5819W; JLCPCB ID (none) -> C134429; Manufacturer (none) -> Diodes Incorporated; Part Number (none) -> B140HW-7; Specifications (none) -> SCHOTTKY RECTIFIER 1.0A 40Vrrm 0.55Vf
- R45, R46: footprint Resistor_THT:R_Axial_DIN0207_L6.3mm_D2.5mm_P7.62mm_Horizontal -> Resistor_SMD:R_0603_1608Metric_Pad0.98x0.95mm_HandSolder
Connections:
- net +12V: now also C23.1, C18.1, U7.3 (VI)
- net +5V: now also C21.1, U7.2 (VO); no longer C23.1
- net -10V_REF: now also C17.1, U6.2 (A)
- net -12V: now also C19.2
- net -3V6_REF: now also DZ1.2 (A)
- net GND: now also C17.2, C18.2, C19.1, C21.2, DZ1.1 (K), U6.1 (K), U7.1 (GND)
Other:
- moved on the sheet: C20
