File: Beaks Pro/Hardware/beaks_pro_8hp/stm32.kicad_sch (KiCad schematic)
At the start: 16 parts, among them J16 Conn_01x20_Socket, J17 Conn_01x20_Socket, Q1 2N3904, Q2 2N3904, U8 Bluepill

Commit message: Layout done on 8HP SMT version
Parts:
- removed Q1, Q2: 2N3904, Package_TO_SOT_THT:TO-92_Inline_Wide, symbol Transistor_BJT:2N3904
- added Q1, Q2: S8050 J3Y, PCM_Package_TO_SOT_SMD_AKL:SOT-23, symbol PCM_Transistor_BJT_AKL:MMSS8050
- R47, R48, R49, R50, R51, R52, R53, R54, R55, R56, R57: footprint Resistor_THT:R_Axial_DIN0207_L6.3mm_D2.5mm_P7.62mm_Horizontal -> Resistor_SMD:R_0603_1608Metric_Pad0.98x0.95mm_HandSolder
Connections:
- net GND: now also Q1.2 (E), Q2.2 (E)
- net STM_TRIG_1: now also Q1.3 (C)
- net STM_TRIG_2: now also Q2.3 (C)
- net at R56.2: now also Q1.1 (B)
- net at R57.2: now also Q2.1 (B)
