File: Beaks Pro/Hardware/andes_8hp/frontpanel/frontpanel.kicad_pcb (KiCad board)
At the start: 2 copper layers, 40.3 x 128.5 mm, 46 parts

Commit message: Properly delete
Other:
- board text removed: "1 - OUT - 2"
