File: Beaks Pro/Hardware/andes_10hp/andes_10HP.kicad_pcb (KiCad board)
At the start: 2 copper layers, 181.5 x 128.5 mm, 157 parts, among them J1 Pins_02x10_P2.54mm_TH, J11 out1, J12 out2, J13 Eurorack Power, J14 Pins_02x10_P2.54mm_TH, J2 Pins_02x10_P2.54mm_TH, J3 CV1, J4 CV2, J5 CV3, J6 CV4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

Commit message: Small updates.
Parts:
- added Ref**: Val**, SVG PCB:DirtNacho, F.Cu at (55.5, 147.7)
Other:
- board text added: "Front Plate designed by Nacho. V0.1"
