File: Andes/Hardware/andes_8hp/front_pcb/front_pcb.kicad_sch (KiCad schematic)
At the start: 30 parts, among them J11 out1, J12 out2, J2 Conn_02x12_Odd_Even, J3 CV1, J4 CV2, J5 CV3, J6 CV4, J7 in1, J8 in2, J9 Conn_02x08_Odd_Even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

Commit message: Fix attenuverter inversion, generate new gerber, update .gitignore
Connections:
- net CV1_JACK: now also RV4.1; no longer RV4.3
- net CV2_JACK: now also RV5.1; no longer RV5.3
- net CV3_JACK: now also RV6.1; no longer RV6.3
- net CV4_JACK: now also RV8.1; no longer RV8.3
- net GND1: now also RV4.3, RV5.3, RV6.3, RV8.3; no longer RV4.1, RV5.1, RV6.1, RV8.1
Changed lines of the file:
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@@
 		(lib_id "Device:R_Potentiometer")
 		(at 45.72 83.82 0)
-		(mirror x)
 		(unit 1)
 		(exclude_from_sim no)
@@
 		(dnp no)
 		(property "Reference" "RV5"
-			(at 43.942 82.6516 0)
+			(at 43.942 84.9884 0)
 			(effects
 				(font
@@
 		)
 		(property "Value" "B100k"
-			(at 43.942 84.963 0)
+			(at 43.942 82.677 0)
 			(effects
 				(font
@@
 		(lib_id "Device:R_Potentiometer")
 		(at 45.72 133.35 0)
-		(mirror x)
 		(unit 1)
 		(exclude_from_sim no)
@@
 		(dnp no)
 		(property "Reference" "RV6"
-			(at 43.942 132.1816 0)
+			(at 43.942 134.5184 0)
 			(effects
 				(font
@@
 		)
 		(property "Value" "B100k"
-			(at 43.942 134.493 0)
+			(at 43.942 132.207 0)
 			(effects
 				(font
@@
 		(lib_id "Device:R_Potentiometer")
 		(at 45.72 34.29 0)
-		(mirror x)
 		(unit 1)
 		(exclude_from_sim no)
@@
 		(dnp no)
 		(property "Reference" "RV4"
-			(at 43.942 33.1216 0)
+			(at 43.942 35.4584 0)
 			(effects
 				(font
@@
 		)
 		(property "Value" "B100k"
-			(at 43.942 35.433 0)
+			(at 43.942 33.147 0)
 			(effects
 				(font
@@
 		(lib_id "Device:R_Potentiometer")
 		(at 115.57 34.29 0)
-		(mirror x)
 		(unit 1)
 		(exclude_from_sim no)
@@
 		(dnp no)
 		(property "Reference" "RV8"
-			(at 113.792 33.1216 0)
+			(at 113.792 35.4584 0)
 			(effects
 				(font
@@
 		)
 		(property "Value" "B100k"
-			(at 113.792 35.433 0)
-			(effects
-				(font
+			(at 113.792 33.147 0)
+			(effects
+				(font
