File: Andes/Hardware/andes_8hp/andes.kicad_pcb (KiCad board)
At the start: 2 copper layers, 40 x 110 mm, 110 parts, among them J1 Conn_02x08_Odd_Even, J13 Eurorack Power, J14 Conn_02x12_Odd_Even, Q1 S8050 J3Y, Q2 S8050 J3Y, U1 TL072CD, U2 MCP6002-I-SN, U3 TL072CD, U4 MCP6002-I-SN, U5 TL074CD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

Commit message: Update Andes 8HP with fixes
Parts:
- R45: value 2k -> 330
- R46: value 10k -> 1k2
Changed lines of the file:
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@@
 			)
 		)
-		(property "Value" "10k"
+		(property "Value" "1k2"
 			(at 0 1.43 0)
 			(layer "F.Fab")
@@
 			)
 		)
-		(property "Value" "2k"
+		(property "Value" "330"
 			(at 0 1.43 90)
 			(layer "F.Fab")
