File: Andes/Hardware/andes_8hp/power.kicad_sch (KiCad schematic)
At the start: 17 parts, among them J13 Eurorack Power, U6 LM4040DBZ-10, U7 AMS1117-5.0

Commit message: Update Andes 8HP with fixes
Parts:
- R45: value 2k -> 330
- R46: value 10k -> 1k2
Changed lines of the file:
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@@
 			)
 		)
-		(property "Value" "10k"
+		(property "Value" "1k2"
 			(at 156.21 113.03 90)
 			(effects
@@
 			)
 		)
-		(property "Value" "2k"
+		(property "Value" "330"
 			(at 95.25 110.49 90)
 			(effects
