File: Andes/Hardware/andes_12hp/andes_12hp.kicad_pcb (KiCad board)
At the start: 2 copper layers, 141 parts, among them J1 Pins_02x10_P2.54mm_TH, J11 out1, J12 out2, J13 Eurorack Power, J14 Pins_02x10_P2.54mm_TH, J2 Pins_02x10_P2.54mm_TH, J3 CV1, J4 CV2, J5 CV3, J6 CV4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

Commit message: Sync changes in 8HP Andes to 12HP Andes
Parts:
- D1: value 3.6 -> BZX55C3V6
- R45: value 2k -> 330R
- R46: value 10k -> 1k5
Connections:
- RV4 pad 1: GND1 -> /Front PCB/CV1_JACK
- RV4 pad 3: /Front PCB/CV1_JACK -> GND1
- RV5 pad 1: GND1 -> /Front PCB/CV2_JACK
- RV5 pad 3: /Front PCB/CV2_JACK -> GND1
- RV6 pad 1: GND1 -> /Front PCB/CV3_JACK
- RV6 pad 3: /Front PCB/CV3_JACK -> GND1
- RV8 pad 1: GND1 -> /Front PCB/CV4_JACK
- RV8 pad 3: /Front PCB/CV4_JACK -> GND1
Changed lines of the file:
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@@
 			(layers "*.Cu" "*.Mask")
 			(remove_unused_layers no)
-			(net 24 "GND1")
+			(net 56 "/Front PCB/CV2_JACK")
 			(pinfunction "1")
 			(pintype "passive")
@@
 			(layers "*.Cu" "*.Mask")
 			(remove_unused_layers no)
-			(net 56 "/Front PCB/CV2_JACK")
+			(net 24 "GND1")
 			(pinfunction "3")
 			(pintype "passive")
@@
 			(layers "*.Cu" "*.Mask")
 			(remove_unused_layers no)
-			(net 24 "GND1")
+			(net 51 "/Front PCB/CV3_JACK")
 			(pinfunction "1")
 			(pintype "passive")
@@
 			(layers "*.Cu" "*.Mask")
 			(remove_unused_layers no)
-			(net 51 "/Front PCB/CV3_JACK")
+			(net 24 "GND1")
 			(pinfunction "3")
 			(pintype "passive")
@@
 			(layers "*.Cu" "*.Mask")
 			(remove_unused_layers no)
-			(net 24 "GND1")
+			(net 55 "/Front PCB/CV1_JACK")
 			(pinfunction "1")
 			(pintype "passive")
@@
 			(layers "*.Cu" "*.Mask")
 			(remove_unused_layers no)
-			(net 55 "/Front PCB/CV1_JACK")
+			(net 24 "GND1")
 			(pinfunction "3")
 			(pintype "passive")
@@
 			)
 		)
-		(property "Value" "10k"
+		(property "Value" "1k5"
 			(at 3.81 2.37 0)
 			(layer "F.Fab")
@@
 			)
 		)
-		(property "Value" "3.6"
+		(property "Value" "BZX55C3V6"
 			(at 3.81 2.12 0)
 			(layer "F.Fab")
@@
 			(layers "*.Cu" "*.Mask")
 			(remove_unused_layers no)
-			(net 24 "GND1")
+			(net 54 "/Front PCB/CV4_JACK")
 			(pinfunction "1")
 			(pintype "passive")
@@
 			(layers "*.Cu" "*.Mask")
 			(remove_unused_layers no)
-			(net 54 "/Front PCB/CV4_JACK")
+			(net 24 "GND1")
 			(pinfunction "3")
 			(pintype "passive")
@@
 			)
 		)
-		(property "Value" "2k"
+		(property "Value" "330R"
 			(at 3.81 2.37 0)
 			(layer "F.Fab")
