File: Andes/Hardware/andes_12hp/front.kicad_sch (KiCad schematic)
At the start: 30 parts, among them J11 out1, J12 out2, J2 Pins_02x10_P2.54mm_TH, J3 CV1, J4 CV2, J5 CV3, J6 CV4, J7 in1, J8 in2, J9 Pins_02x10_P2.54mm_TH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

Commit message: Sync changes in 8HP Andes to 12HP Andes
Connections:
- net CV1_JACK: now also RV4.1; no longer RV4.3
- net CV2_JACK: now also RV5.1; no longer RV5.3
- net CV3_JACK: now also RV6.1; no longer RV6.3
- net CV4_JACK: now also RV8.1; no longer RV8.3
- net GND1: now also RV4.3, RV5.3, RV6.3, RV8.3; no longer RV4.1, RV5.1, RV6.1, RV8.1
