File: Sluisbrinkie Braun/Hardware/PI_SCOPE/PI_SCOPE.kicad_sch (KiCad schematic)
At the start: 97 parts, among them J1 Eurorack Power, J10 CV4, J2 USB_C_Receptacle_USB2.0_16P, J3 CV1, J4 CV2, J5 CV3, J6 CV4, J7 CV1, J8 CV2, J9 CV3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

Commit message: [Braun] Several hardware fixes, move display from SPI1 to SPI0
Parts:
- SW4: value PEC12R-3222F -> PEC11R-3222F; footprint Rotary_Encoder:RotaryEncoder_Alps_EC12E-Switch_Vertical_H20mm -> Rotary_Encoder:RotaryEncoder_Alps_EC11E-Switch_Vertical_H20mm
Connections:
- net CS: now also U8.3 (GPIO1); no longer U8.12 (GPIO9)
- net MOSI: now also U8.5 (GPIO3); no longer U8.14 (GPIO11)
- net SCK: now also U8.4 (GPIO2); no longer U8.13 (GPIO10)
